File: LiPoPoE.sch (KiCad schematic (older format))
At the start: 20 parts

Commit message: Added pdf and others
Parts:
- removed C? (x2): C, symbol C
- added C3, C7: 10uF 50V, Capacitors_SMD:C_0805_HandSoldering, symbol C
- added C6: 220uF 35V, Capacitors_SMD:CP_Elec_8x10.5, symbol CP
- added D10, D3, D4, D5, D6, D7, D8, D9: ESDZL5-1F4, Diodes_SMD:D_0603, symbol D_Zener
- C1: renamed from C?; value CP -> 100uF 35V; footprint (none) -> Capacitors_SMD:CP_Elec_6.3x7.7
- C2: renamed from C?; value C -> 10uF 50V; footprint (none) -> Capacitors_SMD:C_0805_HandSoldering
- C4: renamed from C?; value 50pF -> 50pF 50V; footprint (none) -> Capacitors_SMD:C_0805_HandSoldering
- C5: renamed from C?; value CP -> 220uF 35V; footprint (none) -> Capacitors_SMD:CP_Elec_8x10.5
- D1: renamed from D?; value D_Zener -> SMBJ45A-E3/52; footprint (none) -> footprints:DO-214AA
- D11: renamed from D?; footprint (none) -> Diodes_THT:D_DO-41_SOD81_P2.54mm_Vertical_AnodeUp
- D2: renamed from D?; value D -> 1N4007; footprint (none) -> Diodes_THT:D_DO-41_SOD81_P2.54mm_Vertical_AnodeUp
- J1: renamed from J?; footprint (none) -> Connectors_JST:JST_XH_B02B-XH-A_02x2.50mm_Straight
- J2, J3: renamed from J?; footprint (none) -> Connectors:RJ45_8
- L1: renamed from L?; footprint (none) -> Inductors_SMD:L_Taiyo-Yuden_NR-60xx_HandSoldering
- R1, R2: renamed from R?; value 0 -> 0R00; footprint (none) -> Resistors_SMD:R_0805_HandSoldering
- R3, R4: renamed from R?; footprint (none) -> Resistors_SMD:R_0805_HandSoldering
- R5: renamed from R?; value R -> 20k0; footprint (none) -> Resistors_SMD:R_0805_HandSoldering
- R6: renamed from R?; value R -> 1k10; footprint (none) -> Resistors_SMD:R_0805_HandSoldering
- U1: renamed from U?; footprint (none) -> Housings_DIP:DIP-8_W7.62mm
Connections:
- net +24V: now also C6.1, C7.1
- net GND: now also C3.2, C6.2, C7.2, D3.2 (A), D4.2 (A), D5.2 (A), D6.2 (A)
- net RX+: now also D5.1 (K), D7.1 (K)
- net RX-: now also D6.1 (K), D8.1 (K)
- net TX+: now also D3.1 (K), D9.1 (K)
- net TX-: now also D10.1 (K), D4.1 (K)
- net VCC: now also C3.1
- new net: D7.2 (A), D8.2 (A)
- new net: D10.2 (A), D9.2 (A)
Other:
- note added: "24 Volt Regulator"
- note added: "45V TVS Uni-directional"
- note added: "5.5V TVS Bi-directional"
- note added: "5.5V TVS Uni-directional"
- moved on the sheet: C1, C2, C4, C5, D11, L1, R3, R4, R5, R6, U1
